Commit message: simulated cone detection, reset, and visuals

File: qutms_sim/urdf/lidar.urdf.xacro (robot description, xacro)
@@ -2,5 +2,5 @@
 <robot name="LiDAR" xmlns:xacro="http://www.ros.org/wiki/xacro">
   <xacro:property name="M_PI" value="3.1415926535897931" />
-  <xacro:macro name="LiDAR" params="*origin parent prefix">
+  <xacro:macro name="LiDAR" params="*origin parent prefix namespace">
     <xacro:property name="hz" value="10"/>
     <xacro:property name="samples" value="1000"/>
@@ -65,5 +65,5 @@
         <plugin name="laserscan_plugin" filename="libgazebo_ros_lidar.so">
           <ros>
-            <namespace>/sim</namespace>
+            <namespace>/${prefix}</namespace>
             <remapping>~/out:=scan</remapping>
           </ros>

File: qutms_sim/urdf/robot.urdf.xacro (robot description, xacro)
@@ -6,4 +6,5 @@
     <xacro:arg name="base_frame" default="base_link"/>
     <xacro:arg name="display_car" default="true"/>
+    <!-- <xacro:arg name="namespace" default="sim"/> -->
     <!-- Imports -->
     <xacro:include filename="$(find qutms_sim)/urdf/wheels.urdf.xacro"/>
@@ -11,8 +12,15 @@
     <!--  Gazebo ROS 2 plugins  -->
     <gazebo>
-        <!-- this name also is ROS 2 node name -->
+        <!-- plugin name also is ROS 2 node name -->
         <plugin name="vehicle" filename="libgazebo_vehicle.so"></plugin>
         <ros>
-          <namespace>/sim</namespace>
+          <!-- could make this an arg -->
+          <namespace>/$(arg namespace)</namespace>
+        </ros>
+    </gazebo>
+    <gazebo>
+        <plugin name="cone_detection" filename="libgazebo_cone_detection.so"></plugin>
+        <ros>
+          <namespace>/$(arg namespace)</namespace>
         </ros>
     </gazebo>
@@ -84,5 +92,5 @@
     <xacro:rear_wheel lr_prefix="right" lr_reflect="-1" />
     <!-- LiDAR -->
-    <xacro:LiDAR parent="chassis" prefix="velodyne">
+    <xacro:LiDAR parent="chassis" prefix="velodyne" namespace="$(arg namespace)">
         <origin xyz="1.590 0.0 0.0" rpy="0 0 0"/>
     </xacro:LiDAR>
